File: BLEelectronics/CR2025_Nordic/CR2025_Nordic.sch (KiCad schematic (older format))
At the start: 32 parts, among them IC1 LTC4412xS6, IC2 PCF8523T, IC3 MX25R6435FM2IL0, IC4 LTC4054LES5-4.2#TRPBF, J1 Nordic_nRF52840_breakout, J4 Conn_01x01_Female, Q1 Si2307CDS, U1 LP5907MFX-3.3, U2 BAT-HLD-001, U3 ESD401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

Commit message: refactored the MVP 1a to single sided form factor.
Parts:
- removed FID1, FID2: Fiducial, Fiducial:Fiducial_0.5mm_Mask1mm, symbol Mechanical:Fiducial
- removed H1: MountingHole, MountingHole:MountingHole_2.2mm_M2_Pad, symbol Mechanical:MountingHole
- removed J4: Conn_01x01_Female, Connector_PinHeader_2.54mm:PinHeader_1x01_P2.54mm_Vertical, symbol Connector:Conn_01x01_Female
- removed R1, R2, R3, R5, R7: 0, Resistor_SMD:R_0603_1608Metric_Pad1.05x0.95mm_HandSolder, symbol Device:R
- added JP1, JP2: Jumper_2_Open, Jumper:SolderJumper-2_P1.3mm_Open_RoundedPad1.0x1.5mm, symbol Jumper:Jumper_2_Open
Connections:
- wire segments 69 -> 67
- no-connect marks 11 -> 12
Other:
- moved on the sheet: C3, D4, IC4, R6
