File: BLEelectronics/ble_mvp_1B-rev0/ble_covid_opensource_hw.kicad_pcb (KiCad board)
At the start: 2 copper layers, 34.3 x 28.3 mm, 76 parts, among them IC1 LTC4412xS6, IC2 LTC4054LES5-4.2#TRPBF, IC3 PCF8523T, IC4 MX25R6435FM2IL0, J1 USB_B_Micro, J3 Conn_02x05_Odd_Even, Q1 Si2307CDS, SW1 NO, SW2 SW_MEC_5G, U1 BAT-HLD-001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

Commit message: renamed files in mvp1a-rev0 folder, added schematic and gerber pdfs
Parts:
- removed C19: N.C., Capacitor_SMD:C_0201_0603Metric
- removed FID1, FID2, FID3: Fiducial, Fiducial:Fiducial_0.5mm_Mask1mm
- removed H1: MountingHole, MountingHole:MountingHole_2.2mm_M2_DIN965_Pad
- removed R1: 0, Resistor_SMD:R_0603_1608Metric_Pad1.05x0.95mm_HandSolder
- removed R4: 0, Resistor_SMD:R_0402_1005Metric
- added JP2: Jumper_NO_Small, Jumper:SolderJumper-2_P1.3mm_Open_RoundedPad1.0x1.5mm, F.Cu at (145.3, 74.4)
- added JP3: Jumper_NO_Small, Jumper:SolderJumper-2_P1.3mm_Open_RoundedPad1.0x1.5mm, F.Cu at (151.6, 66.4)
- C16, C31: value 100nF -> 0.01uF
- C3, C5: footprint Capacitor_SMD:C_0603_1608Metric_Pad1.05x0.95mm_HandSolder -> Capacitor_SMD:C_0402_1005Metric
- C30: value 100nF -> 0.1uF
- R2: footprint Resistor_SMD:R_0603_1608Metric_Pad1.05x0.95mm_HandSolder -> Resistor_SMD:R_0603_1608Metric
- R8: value 1k2 -> 1K2
- R9: value 2k2 -> 2K2
- moved C3 4.00 mm to (159.0, 75.9), turned to 90 degrees
- moved C5 0.85 mm to (146.3, 79.1), turned to 0 degrees
- moved C18 0.82 mm to (138.3, 94.4)
- moved C2 0.72 mm to (142.6, 75.0)
- moved C4 0.72 mm to (142.3, 81.1)
- moved C15 0.30 mm to (139.5, 92.8)
- moved R5 0.17 mm to (159.4, 93.3)
- moved R6 0.16 mm to (159.4, 95.8)
- moved C28 0.13 mm to (143.4, 86.2)
- turned C1 to 270 degrees
Connections:
- C1 pad 1: /3V -> GND
- C1 pad 2: GND -> /3V
- C5 pad 1: /VDD_3V -> GND
- C5 pad 2: GND -> /VDD_3V
Routing:
- net /D-: track 4.63 -> 19.7 mm, vias 0 -> 2
- net /VDD_3V: track 142.2 -> 127.2 mm, vias 2 -> 4
- net /D+: track 7.40 -> 18.9 mm, vias 0 -> 2
- net /SCLK: track 1.91 -> 12.7 mm
- net /WP: track 11.1 -> 20.9 mm
- net /3V: track 57.4 -> 50.1 mm
- net /SI: track 6.73 -> 13.9 mm
- net GND: track 158.8 -> 163.4 mm, vias 16 -> 17
- net Net-(IC3-Pad2): track 0.00 -> 2.81 mm
- net Net-(IC3-Pad1): track 0.00 -> 2.80 mm
- net /5Vusb: track 15.3 -> 16.9 mm
- net Net-(C3-Pad1): track 17.3 -> 15.7 mm
- net Net-(C24-Pad1): track 17.1 -> 16.1 mm
- net Net-(C4-Pad2): track 4.61 -> 3.78 mm
- net Net-(C18-Pad2): track 3.68 -> 2.88 mm
Other:
- board size 34.3 x 28.3 mm -> 36 x 28.3 mm
