File: BLEelectronics/ble_mvp_1B-rev0/ble_covid_opensource_hw.sch (KiCad schematic (older format))
At the start: 36 parts, among them IC1 LTC4412xS6, IC2 LTC4054LES5-4.2#TRPBF, IC3 PCF8523T, IC4 MX25R6435FM2IL0, J1 USB_B_Micro, Q1 Si2307CDS, U1 BAT-HLD-001, U2 ESD401, U3 ESD401, U4 LP5907MFX-3.3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

Commit message: renamed files in mvp1a-rev0 folder, added schematic and gerber pdfs
Parts:
- removed FID1, FID2, FID3: Fiducial, Fiducial:Fiducial_0.5mm_Mask1mm, symbol Mechanical:Fiducial
- removed H1: MountingHole, MountingHole:MountingHole_2.2mm_M2_DIN965_Pad, symbol Mechanical:MountingHole
- removed R1: 0, Resistor_SMD:R_0603_1608Metric_Pad1.05x0.95mm_HandSolder, symbol Device:R
- removed R4: 0, Resistor_SMD:R_0402_1005Metric, symbol Device:R
- added JP2, JP3: Jumper_NO_Small, Jumper:SolderJumper-2_P1.3mm_Open_RoundedPad1.0x1.5mm, symbol Device:Jumper_NO_Small
- C1: DPN 311-1344-2-ND -> 490-10701-1-ND; MFR Yageo -> Murata Electronics; MPN CC0603KRX7R9BB104 -> GRM155R71H104ME14D
- C2: DPN (none) -> 1276-1067-2-ND; MFR (none) -> Samsung Electro-Mechanics; MPN (none) -> CL05A105KO5NNNC
- C3: footprint Capacitor_SMD:C_0603_1608Metric_Pad1.05x0.95mm_HandSolder -> Capacitor_SMD:C_0402_1005Metric; DPN 1276-1862-1-ND -> 1276-1067-2-ND; MFR Samsung -> Samsung Electro-Mechanics; MPN CL10A105KO5LNNC -> CL05A105KO5NNNC
- C4: DPN 1276-1862-1-ND -> 1276-1067-2-ND; MFR (none) -> Samsung Electro-Mechanics; MPN (none) -> CL05A105KO5NNNC
- C5: footprint Capacitor_SMD:C_0603_1608Metric_Pad1.05x0.95mm_HandSolder -> Capacitor_SMD:C_0402_1005Metric; DPN 311-1344-2-ND -> 490-10701-1-ND; MFR Yageo -> Murata Electronics; MPN CC0603KRX7R9BB104 -> GRM155R71H104ME14D
- C8, C9: DPN 311-1344-2-ND -> 311-3567-1-ND; MPN CC0603KRX7R9BB104 -> CC0603KPX7R9BB104
- D3, J1, X3: LCSCPN (none) -> -; SIM (none) -> -; SPN (none) -> -; SPR (none) -> -
- FB1, FB2: DPN (none) -> -; LCSCPN (none) -> -; SIM (none) -> -; SPN (none) -> -; SPR (none) -> -
- R2: footprint Resistor_SMD:R_0603_1608Metric_Pad1.05x0.95mm_HandSolder -> Resistor_SMD:R_0603_1608Metric; DPN RC0201FR-071K69L -> 311-560KGRCT-ND; MPN RC0201FR-07560KL -> RC0603JR-07560KL
- R3: DPN (none) -> YAG3044CT-ND; MFR (none) -> Yageo; MPN (none) -> RC0402FR-071K69L
- R5, R6: DPN 311-4.70KHRCT-ND -> 311-10KJRCT-ND; MPN RC0603FR-074K7L -> RC0402JR-0710KL
Connections:
- net 3V: now also C1.2, JP3.2; no longer C1.1
- net 5Vusb: now also JP2.1
- net GND: now also C1.1, C5.1; no longer C1.2, C5.2
- net VDD_3V: now also C5.2; no longer C5.1
- net at C3.1, IC2.4 (VCC): now also JP2.2
- net at D2.1 (K): now also JP3.1
