File: BLEelectronics/ble_mvp_1A-rev1/ble_mvp_1A-rev1.sch (KiCad schematic (older format))
At the start: 25 parts, among them IC1 LTC4412xS6, IC2 PCF8523T, IC3 MX25R6435FM2IL0, IC4 LTC4054LES5-4.2#TRPBF, J1 Nordic_nRF52840_breakout, Q1 Si2307CDS, U1 LP5907MFX-3.3, U2 BAT-HLD-001, U3 ESD401, U4 ESD401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

Commit message: correct CS to CS# in schematic and pdfs for all mvps
Connections:
- net labels added: CS#
- net labels removed: CS
Other:
- note added: "NB: CS# uses inverted logic"
- note removed: "Confirmed no pull-up/down\nresistors for SPI protocol\nAdd 100nF cap between \nGND and VCC"
Changed lines of the file:
@@
 RESET
 Text Label 8750 4000 2    50   ~ 0
-CS
+CS#
 Text Label 5300 1600 2    50   ~ 0
 SO
 Text Label 5300 1500 2    50   ~ 0
-CS
+CS#
 Text Label 5300 1900 2    50   ~ 0
 SI
@@
 Text Label 8750 4200 2    50   ~ 0
 WP
-Text Notes 4000 1700 0    50   ~ 0
-Confirmed no pull-up/down\nresistors for SPI protocol\nAdd 100nF cap between \nGND and VCC
 Text Label 6650 3650 0    50   ~ 0
 VDD_3V
@@
 NoConn ~ 8650 2350
 NoConn ~ 7950 4250
+Text Notes 8550 4950 0    50   ~ 0
+NB: CS# uses inverted logic
 $EndSCHEMATC

Commit message: Additional changes to schematic labelling.
Connections:
- net labels added: ~CS~, ~RESET~, ~WP~
- net labels removed: CS#, RESET, WP
Other:
- note added: "NB: ~CS~ ~WP~ ~RESET~ use inverted logic"
- note added: "~CS~ - P0.17\nCLK - P0.19\nSI - P0.20\nSO - P0.21\n~WP~ - P0.22\n~RESET~ (SIO3 - pin7) - P0.23\nPinouts from development board schematic\n"
- note removed: "CS - P0.17\nCLK - P0.19\nSI - P0.20\nSO - P0.21\nWP - P0.22\nSIO3/HOLD/RESET(pin7) - P0.23\nPinouts from development board schematic\n"
- note removed: "NB: CS# uses inverted logic"
Changed lines of the file:
@@
 SO
 Text Label 10400 4100 0    50   ~ 0
-RESET
+~RESET~
 Text Label 8750 4000 2    50   ~ 0
-CS#
+~CS~
 Text Label 5300 1600 2    50   ~ 0
 SO
 Text Label 5300 1500 2    50   ~ 0
-CS#
+~CS~
 Text Label 5300 1900 2    50   ~ 0
 SI
@@
 P1.15 is a low frequency GPIO (<10kHz)
 Text Label 5300 1800 2    50   ~ 0
-WP
+~WP~
 Text Label 8750 4200 2    50   ~ 0
-WP
+~WP~
 Text Label 6650 3650 0    50   ~ 0
 VDD_3V
@@
 TVS diode \nfor ESD\nprotection
 Text Label 5300 2000 2    50   ~ 0
-RESET
+~RESET~
 Text Notes 3950 2750 0    50   ~ 0
-CS - P0.17\nCLK - P0.19\nSI - P0.20\nSO - P0.21\nWP - P0.22\nSIO3/HOLD/RESET(pin7) - P0.23\nPinouts from development board schematic\n
+~CS~ - P0.17\nCLK - P0.19\nSI - P0.20\nSO - P0.21\n~WP~ - P0.22\n~RESET~ (SIO3 - pin7) - P0.23\nPinouts from development board schematic\n
 Text Notes 6700 3450 0    50   ~ 0
 VDD powers chip. VBat is for time \nkeeping backup with switching logic.
@@
 NoConn ~ 7950 4250
 Text Notes 8550 4950 0    50   ~ 0
-NB: CS# uses inverted logic
+NB: ~CS~ ~WP~ ~RESET~ use inverted logic
 $EndSCHEMATC
