File: BLEelectronics/uBit_carrier/uBit_carrier.sch (KiCad schematic (older format))
At the start: 14 parts, among them J1 microbit_edge_connector, J2 Conn_01x02_Male, J3 Micro_SD_Card_Det_Hirose_DM3AT, U1 W25Q128JV, U2 MCP1253-ADJI_MS

Commit message: BOM clean, pdf generated, rev0 submitted to JLCPCB
Parts:
- C2, C3, C5: LCSCPN C385893 -> C29936
- C4, C6: LCSCPN C126586 -> C15850
- R1: LCSCPN C234322 -> C22819
- R2: LCSCPN C209220 -> C25804
- R3: LCSCPN C269682 -> C25803
- U1: DPN (none) -> W25Q128JVSIQ-ND
Other:
- note added: "DI"
- note added: "DO"
